Commit message: simulator: changed fusion project joints

File: src/AGV_simulator_description/urdf/AGV_simulator.xacro (robot description, xacro)
@@ -24,3 +24,107 @@
   </collision>
 </link>
+<link name="front_left_1_1_1_1">
+  <inertial>
+    <origin xyz="4.163336342344337e-17 -0.03900000000000001 0.0" rpy="0 0 0"/>
+    <mass value="19.2359718179303"/>
+    <inertia ixx="0.057843" iyy="0.09618" izz="0.057843" ixy="-0.0" iyz="-0.0" ixz="0.0"/>
+  </inertial>
+  <visual>
+    <origin xyz="-0.103 0.02 -0.07" rpy="0 0 0"/>
+    <geometry>
+      <mesh filename="file://$(find AGV_simulator_description)/meshes/front_left_1_1_1_1.stl" scale="0.001 0.001 0.001"/>
+    </geometry>
+    <material name="silver"/>
+  </visual>
+  <collision>
+    <origin xyz="-0.103 0.02 -0.07" rpy="0 0 0"/>
+    <geometry>
+      <mesh filename="file://$(find AGV_simulator_description)/meshes/front_left_1_1_1_1.stl" scale="0.001 0.001 0.001"/>
+    </geometry>
+  </collision>
+</link>
+<link name="back_left_1_1_1_1">
+  <inertial>
+    <origin xyz="1.1102230246251565e-16 -0.03899999999999999 0.0" rpy="0 0 0"/>
+    <mass value="19.2359718179303"/>
+    <inertia ixx="0.057843" iyy="0.09618" izz="0.057843" ixy="-0.0" iyz="-0.0" ixz="0.0"/>
+  </inertial>
+  <visual>
+    <origin xyz="-0.777 0.02 -0.07" rpy="0 0 0"/>
+    <geometry>
+      <mesh filename="file://$(find AGV_simulator_description)/meshes/back_left_1_1_1_1.stl" scale="0.001 0.001 0.001"/>
+    </geometry>
+    <material name="silver"/>
+  </visual>
+  <collision>
+    <origin xyz="-0.777 0.02 -0.07" rpy="0 0 0"/>
+    <geometry>
+      <mesh filename="file://$(find AGV_simulator_description)/meshes/back_left_1_1_1_1.stl" scale="0.001 0.001 0.001"/>
+    </geometry>
+  </collision>
+</link>
+<link name="back_right_1_1_1_1">
+  <inertial>
+    <origin xyz="-1.73673033732058e-08 0.039000000000000146 -1.5646219458931299e-09" rpy="0 0 0"/>
+    <mass value="19.2359718179303"/>
+    <inertia ixx="0.057843" iyy="0.09618" izz="0.057843" ixy="0.0" iyz="0.0" ixz="0.0"/>
+  </inertial>
+  <visual>
+    <origin xyz="-0.777 -0.58 -0.07" rpy="0 0 0"/>
+    <geometry>
+      <mesh filename="file://$(find AGV_simulator_description)/meshes/back_right_1_1_1_1.stl" scale="0.001 0.001 0.001"/>
+    </geometry>
+    <material name="silver"/>
+  </visual>
+  <collision>
+    <origin xyz="-0.777 -0.58 -0.07" rpy="0 0 0"/>
+    <geometry>
+      <mesh filename="file://$(find AGV_simulator_description)/meshes/back_right_1_1_1_1.stl" scale="0.001 0.001 0.001"/>
+    </geometry>
+  </collision>
+</link>
+<link name="front_right_1_1_1_1">
+  <inertial>
+    <origin xyz="1.5348196047426654e-09 0.039000000000000035 1.0430812741324402e-09" rpy="0 0 0"/>
+    <mass value="19.235971817930288"/>
+    <inertia ixx="0.057843" iyy="0.09618" izz="0.057843" ixy="0.0" iyz="0.0" ixz="0.0"/>
+  </inertial>
+  <visual>
+    <origin xyz="-0.103 -0.58 -0.07" rpy="0 0 0"/>
+    <geometry>
+      <mesh filename="file://$(find AGV_simulator_description)/meshes/front_right_1_1_1_1.stl" scale="0.001 0.001 0.001"/>
+    </geometry>
+    <material name="silver"/>
+  </visual>
+  <collision>
+    <origin xyz="-0.103 -0.58 -0.07" rpy="0 0 0"/>
+    <geometry>
+      <mesh filename="file://$(find AGV_simulator_description)/meshes/front_right_1_1_1_1.stl" scale="0.001 0.001 0.001"/>
+    </geometry>
+  </collision>
+</link>
+<joint name="Revolute 17" type="continuous">
+  <origin xyz="0.103 -0.02 0.07" rpy="0 0 0"/>
+  <parent link="base_link"/>
+  <child link="front_left_1_1_1_1"/>
+  <axis xyz="0.0 -1.0 0.0"/>
+</joint>
+<joint name="Revolute 18" type="continuous">
+  <origin xyz="0.777 -0.02 0.07" rpy="0 0 0"/>
+  <parent link="base_link"/>
+  <child link="back_left_1_1_1_1"/>
+  <axis xyz="0.0 -1.0 0.0"/>
+</joint>
+<joint name="Revolute 19" type="continuous">
+  <origin xyz="0.777 0.58 0.07" rpy="0 0 0"/>
+  <parent link="base_link"/>
+  <child link="back_right_1_1_1_1"/>
+  <axis xyz="0.0 1.0 0.0"/>
+</joint>
+<joint name="Revolute 20" type="continuous">
+  <origin xyz="0.103 0.58 0.07" rpy="0 0 0"/>
+  <parent link="base_link"/>
+  <child link="front_right_1_1_1_1"/>
+  <axis xyz="0.0 1.0 0.0"/>
+</joint>
 </robot>
